Commit message: Add files via upload

File: urdf/matrix_true_description.urdf (robot description, URDF)
Before this commit: robot matrix_true_description, 17 links, 16 joints
Links:
- link base_link: mass 95.4830322905057 -> 95.483
- link caster_arm_fl_link: mass 0.0228689686367412 -> 0.0228689686598223
- link caster_arm_fr_link: mass 0.0228689686633764 -> 0.0228689686598222
- link caster_arm_rl_link: mass 0.0228689686598223 -> 0.0228689686598218
- link caster_arm_rr_link: mass 0.0228689686367412 -> 0.0228689686598225
- link caster_wheel_rr_link: mass 0.0372150073615412 -> 0.037215
- link depth_cam_mount_point_link: mass 0.0364722860415581 -> 0.0364722860415582
- link imu_link: mass 0.00098313018365204 -> 0.000983130183652039
- link lidar_merged_link: mass 0.0479836298060718 -> 0.0479836298060696
- link ultrasonic_fl_link: mass 0 -> 0.00277452811002928
- link wheel_left_link: mass 1.2499 -> 1.24985940735749
Joints:
- joint caster_arm_fl_joint: origin xyz=0.175 0.1 0.069116 rpy=0 0 0 -> xyz=0.174999999999999 0.100000000000001 0.069116 rpy=0 0 0
- joint caster_arm_fr_joint: origin xyz=0.175 -0.1 0.069116 rpy=0 0 0 -> xyz=0.175000000000001 -0.0999999999999988 0.069116 rpy=0 0 0
- joint caster_arm_rl_joint: origin xyz=-0.175 0.1 0.069116 rpy=0 0 0 -> xyz=-0.175000000000001 0.0999999999999989 0.069116 rpy=0 0 0
- joint caster_arm_rr_joint: origin xyz=-0.175 -0.1 0.069116 rpy=0 0 0 -> xyz=-0.174999999999999 -0.100000000000001 0.069116 rpy=0 0 0
- joint caster_wheel_fl_joint: axis 0 0 1 -> 0 1 0; origin xyz=0 0 0 rpy=0 0 0 -> xyz=-0.0249999999999994 0 -0.0439999999999999 rpy=0 1.5707963267949 0
- joint depth_cam_mount_point_joint: origin xyz=0.14565 0 0.48012 rpy=0 0 0 -> xyz=0.145649999999998 0 0.480116 rpy=0 0 0
- joint imu_joint: origin xyz=-0.02 0 0.34712 rpy=0 0 0 -> xyz=-0.020000000000002 0 0.347116 rpy=0 0 0
- joint lidar_merged_joint: origin xyz=0.155 0 0.29572 rpy=0 0 0 -> xyz=0.155000000000003 0 0.295715793055286 rpy=0 0 3.14159265358979
- joint ultrasonic_fc_joint: origin xyz=0.21264 0 0.23385 rpy=0 0.018394 0 -> xyz=0.212644504488986 0 0.2338466055562 rpy=0 0.0183935250864792 0
- joint ultrasonic_fr_joint: origin xyz=0.16952 -0.1681 0.23408 rpy=0 0.001995 -0.71728 -> xyz=0.169517824893003 -0.168095327438868 0.234077654834356 rpy=0 0.00199498585800991 -0.717281737993582
- joint wheel_left_right: origin xyz=0.0037081 0.2171 0.085 rpy=0 1.5708 0 -> xyz=0.0037081011988188 0.2171 0.0850001069853643 rpy=0 1.5707963267949 0
- joint wheel_right_joint: origin xyz=0.0037081 -0.2171 0.085 rpy=0 1.5708 0 -> xyz=0.00370810119881812 -0.2171 0.0850001069853645 rpy=0 1.5707963267949 0

Commit message: Add files via upload

File: urdf/matrix_true_description.urdf (robot description, URDF)
Before this commit: robot matrix_true_description, 17 links, 16 joints
Links:
- added link rear_camera_link, mass 0.12773; collision mesh filename=package://matrix_true_description/meshes/rear_camera_link.S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; visual mesh filename=package://matrix_true_description/meshes/rear_camera_link.S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
- link base_link: mass 95.483 -> 95.4830322905057
- link caster_arm_fl_link: mass 0.0228689686598223 -> 0.022869
- link caster_arm_fr_link: mass 0.0228689686598222 -> 0.022869
- link caster_arm_rl_link: mass 0.0228689686598218 -> 0.022869
- link caster_arm_rr_link: mass 0.0228689686598225 -> 0.022869
- link caster_wheel_fl_link: mass 0.0372150073615411 -> 0.037215
- link caster_wheel_fr_link: mass 0.0372150073615411 -> 0.037215
- link caster_wheel_rl_link: mass 0.0372150073615412 -> 0.037215
- link depth_cam_mount_point_link: mass 0.0364722860415582 -> 0.036472
- link imu_link: mass 0.000983130183652039 -> 0.00098313
- link lidar_merged_link: mass 0.0479836298060696 -> 0.047984
- link ultrasonic_fc_link: mass 0.00277452812571776 -> 0.0027745
- link ultrasonic_fl_link: mass 0.00277452811002928 -> 0.0027745
- link ultrasonic_fr_link: mass 0.00277452811002927 -> 0.0027745
- link wheel_left_link: mass 1.24985940735749 -> 1.2499
Joints:
- added joint rear_camera_joint: type fixed, parent base_link, child rear_camera_link, origin xyz=-0.111753499872574 0 0.041116 rpy=0 0 -3.14159265358979, axis 0 0 0
